Commit message: adding in spot support

File: software/rpl-unitree-ros/xacro/go1.xacro (robot description, xacro)
@@ -2,4 +2,6 @@
 <robot name="go1" xmlns:xacro="http://www.ros.org/wiki/xacro">
     <xacro:arg name="DEBUG" default="false"/>
+    <xacro:arg name="lidar_height" default="0.2"/>
+    <xacro:arg name="camera_" default="0.2"/>
     <xacro:include filename="$(find go1_description)/xacro/const.xacro"/>
     <xacro:include filename="$(find go1_description)/xacro/materials.xacro"/>
@@ -10,5 +12,9 @@
     <xacro:include filename="$(find go1_description)/xacro/ultraSound.xacro"/>
     <xacro:include filename="$(find rpl-unitree-ros)/xacro/lidar.urdf.xacro"/>
+    <xacro:LIDAR-Settings parent="base" x="0" y="0" z="0.2" >
+    </xacro:LIDAR-Settings>
     <xacro:include filename="$(find rpl-unitree-ros)/xacro/rgbd_camera.urdf.xacro"/>
+    <xacro:RGBDCamera-Settings parent="base" x="0.1" y="0" z="0.15" >
+    </xacro:RGBDCamera-Settings>
     <!-- <xacro:include filename="$(find go1_gazebo)/launch/stairs.urdf.xacro"/> -->
     <!-- <xacro:stairs stairs="15" xpos="0" ypos="0" zpos="0" /> -->

File: software/rpl-unitree-ros/xacro/lidar.urdf.xacro (robot description, xacro)
@@ -1,6 +1,8 @@
-<robot xmlns:xacro="http://www.ros.org/wiki/xacro" name="example">
+<robot xmlns:xacro="http://www.ros.org/wiki/xacro" name="LIDAR-Settings">
+  <xacro:macro name="LIDAR-Settings" params="x:=0 y:=0 z:=0.2 parent:=base">
   <xacro:include filename="$(find velodyne_description)/urdf/VLP-16.urdf.xacro"/>
-  <xacro:VLP-16 parent="base" name="velodyne" topic="/velodyne_points" hz="5" samples="350" min_range="0.1" organize_cloud="true">
-    <origin xyz="0 0 0.2" rpy="0 0 0" />
+  <xacro:VLP-16 parent="${parent}" name="velodyne" topic="/velodyne_points" hz="5" samples="350" min_range="0.1" organize_cloud="true">
+    <origin xyz="${x} ${y} ${z}" rpy="0 0 0" />
   </xacro:VLP-16>
+  </xacro:macro>
 </robot>

File: software/rpl-unitree-ros/xacro/rgbd_camera.urdf.xacro (robot description, xacro)
@@ -1,3 +1,4 @@
-<robot xmlns:xacro="http://www.ros.org/wiki/xacro" name="example">
+<robot xmlns:xacro="http://www.ros.org/wiki/xacro" name="RGBDCamera-Settings">
+  <xacro:macro name="RGBDCamera-Settings" params="x:=0.05 y:=0 z:=0.15 parent:=base">
   <link name="camera">
     <collision>
@@ -10,5 +11,5 @@
       <origin xyz="0 0 0" rpy="0 0 0"/>
       <geometry>
-        <box size="0.001 0.001 0.001"/>
+        <box size="0.01 0.01 0.01"/>
       </geometry>
     </visual>
@@ -20,6 +21,6 @@
   </link>
   <joint name="floating_base_to_camera" type="fixed">
-      <origin rpy="0 0 0" xyz="0.2 0 0.15"/>
-      <parent link="base"/>
+      <origin rpy="0 0 0" xyz="${x} ${y} ${z}"/>
+      <parent link="${parent}"/>
       <child link="camera"/>
   </joint>
@@ -59,3 +60,4 @@
     </sensor>
   </gazebo>
+  </xacro:macro>
 </robot>

Commit message: adding some glue

File: software/rpl-unitree-ros/xacro/go1.xacro (robot description, xacro)
@@ -3,4 +3,6 @@
     <xacro:arg name="DEBUG" default="false"/>
     <xacro:arg name="lidar_height" default="0.2"/>
+    <xacro:arg name="lidar_ry" default="{15/180 * pi}"/>
+    <xacro:arg name="name" default="velodyne"/>
     <xacro:arg name="camera_" default="0.2"/>
     <xacro:include filename="$(find go1_description)/xacro/const.xacro"/>
@@ -12,5 +14,5 @@
     <xacro:include filename="$(find go1_description)/xacro/ultraSound.xacro"/>
     <xacro:include filename="$(find rpl-unitree-ros)/xacro/lidar.urdf.xacro"/>
-    <xacro:LIDAR-Settings parent="base" x="0" y="0" z="0.2" >
+    <xacro:LIDAR-Settings parent="base" name="$(arg name)" ry="$(arg lidar_ry)" z="$(arg lidar_height)" >
     </xacro:LIDAR-Settings>
     <xacro:include filename="$(find rpl-unitree-ros)/xacro/rgbd_camera.urdf.xacro"/>

File: software/rpl-unitree-ros/xacro/lidar.urdf.xacro (robot description, xacro)
@@ -1,7 +1,7 @@
 <robot xmlns:xacro="http://www.ros.org/wiki/xacro" name="LIDAR-Settings">
-  <xacro:macro name="LIDAR-Settings" params="x:=0 y:=0 z:=0.2 parent:=base">
+  <xacro:macro name="LIDAR-Settings" params="x:=0 y:=0 z:=0.2 rx:=0 ry:=0 rz:=0 parent:=base name:=velodyne">
   <xacro:include filename="$(find velodyne_description)/urdf/VLP-16.urdf.xacro"/>
-  <xacro:VLP-16 parent="${parent}" name="velodyne" topic="/velodyne_points" hz="5" samples="350" min_range="0.1" organize_cloud="true">
-    <origin xyz="${x} ${y} ${z}" rpy="0 0 0" />
+  <xacro:VLP-16 parent="${parent}" name="${name}" topic="/velodyne_points" hz="5" samples="350" min_range="0.1" organize_cloud="true">
+    <origin xyz="${x} ${y} ${z}" rpy="${rx} ${ry} ${rz}" />
   </xacro:VLP-16>
   </xacro:macro>
